File: tray-board/hydroponics_tray_controller/hydroponics_tray_controller.kicad_pcb (KiCad board)
At the start: 2 copper layers, 99.5 x 99.5 mm, 29 parts, among them J1 Jumper, J2 Display_Connector, J4 Power_Comms, J5 i2c_Peripherals, J6 1Wire_Peripherals, SW1 RotaryEncoder_Switch, U1 ESP32, U2 SP3485EN, U3 AMS1117-3.3

Commit message: tray-board: replace ST7789 display connector with ILI9341 touch + SD card
J2 is now a 14-pin header matching the actual ILI9341/XPT2046 touch
display (VCC, GND, CS, RESET, DC, MOSI, SCK, LED, MISO, T_CLK, T_CS,
T_DIN, T_DO, T_IRQ), replacing the old 8-pin no-touch ST7789 wiring.
Added J3, a separate 4-pin SD card connector sharing the display SPI
bus with its own CS line. New signals use previously-unused ESP32
GPIOs 14, 19, 34, 35. Verified via KiCad 10 ERC and netlist export.

PCB footprints synced from the updated schematic (Update PCB from
Schematic) - placement and routing for the new pins still needed.

README updated with the corrected display spec and pin list.

Co-Authored-By: Claude Sonnet 5 <noreply@anthropic.com>
Claude-Session: https://claude.ai/code/session_01QYbZEgBzGJ6rSai1ie8nG1
Parts:
- added J3: SD_Connector, Connector_PinHeader_2.54mm:PinHeader_1x04_P2.54mm_Vertical, F.Cu at (86.8, 46.8)
- J2: value Display_Connector -> Display_Connector_Touch; footprint Connector_PinHeader_2.54mm:PinHeader_1x08_P2.54mm_Vertical -> Connector_PinHeader_2.54mm:PinHeader_1x14_P2.54mm_Vertical
- moved J2 11.5 mm to (31.5, 70.5)
- moved C6 4.50 mm to (69.3, 83.2)
- moved C7 4.50 mm to (69.5, 78.2)
- moved R6 4.50 mm to (46.3, 85.8)
- moved R7 4.50 mm to (46.3, 82.2)
- moved R8 4.50 mm to (46.3, 78.2)
- moved SW1 4.50 mm to (64.8, 83.2)
Connections:
- J2 pad 1: GND -> +3V3
- J2 pad 2: +3V3 -> GND
- J2 pad 3: /ESP32_D18 -> /ESP32_D5
- J2 pad 4: /ESP32_D23 -> /ESP32_D4
- J2 pad 5: /ESP32_D4 -> /ESP32_D2
- J2 pad 6: /ESP32_D2 -> /ESP32_D23
- J2 pad 7: /ESP32_D5 -> /ESP32_D18
- U1 pad 10: unconnected-(U1-D14-Pad10) -> /ESP32_D14
- U1 pad 19: unconnected-(U1-D19-Pad19) -> /ESP32_D19
- U1 pad 22: unconnected-(U1-D35-Pad22) -> /ESP32_D35
- U1 pad 24: unconnected-(U1-D34-Pad24) -> /ESP32_D34
- U1 pad 3: GND -> unconnected-(U1-GND-Pad3)
- U1 pad 30: unconnected-(U1-EN-Pad30) -> (no net)
Routing:
- net GND: track 286.7 -> 284.5 mm
- net unconnected-(U1-GND-Pad3): track 0.00 -> 2.22 mm
