File: reservoir-board/hydroponics_reservoir_controller/hydroponics_reservoir_controller.kicad_pcb (KiCad board)
At the start: 2 copper layers, 100 x 100 mm, 82 parts, among them J1 Jumper, Q1 AO3400A, Q2 AO3400A, Q3 AO3400A, Q4 AO3400A, Q5 AO3400A, Q6 AO3400A, Q7 AO3400A, Q8 AO3400A, U1 ESP32, U2 SP3485EN, U3 AMS1117-3.3, U4 TPS54302

Commit message: Add sensor-board KiCad project; reservoir board pin silkscreen
- sensor-board: new KiCad project (schematic + PCB) with 4/5/6-pin
  sensor connector sockets
- reservoir-board: add connector pin labels to silkscreen

Co-Authored-By: Claude Opus 5.5 <noreply@anthropic.com>
Other:
- board text added: "A"
- board text added: "B"
- board text added: "D"
- board text added: "E"
- board text added: "G"
- board text added: "T"
- board text added: "V"
Changed lines of the file:
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@@
 		(tags "connector JST XH vertical")
 		(property "Reference" "1Wire"
-			(at 2.5 -3.55 0)
+			(at 2.4 -6.1 0)
 			(layer "F.SilkS")
 			(effects
@@
 		(tags "connector JST XH vertical")
 		(property "Reference" "Trays"
-			(at 3.75 -3.55 0)
+			(at 3.9 -6.1 0)
 			(layer "F.SilkS")
 			(effects
@@
 		(tags "connector JST XH vertical")
 		(property "Reference" "Level Sensor"
-			(at 3.75 -3.55 0)
+			(at 4 -6.1 0)
 			(layer "F.SilkS")
 			(effects
@@
 		)
 	)
+	(gr_text "V"
+		(at 107.310305 56.463729 90)
+		(layer "F.SilkS")
+		(effects
+			(font
+				(size 1 1)
+				(thickness 0.1)
+			)
+			(justify left bottom)
+		)
+	)
+	(gr_text "B"
+		(at 109.810305 56.463729 90)
+		(layer "F.SilkS")
+		(effects
+			(font
+				(size 1 1)
+				(thickness 0.1)
+			)
+			(justify left bottom)
+		)
+	)
+	(gr_text "A"
+		(at 112.310305 56.463729 90)
+		(layer "F.SilkS")
+		(effects
+			(font
+				(size 1 1)
+				(thickness 0.1)
+			)
+			(justify left bottom)
+		)
+	)
+	(gr_text "G"
+		(at 116.310305 56.463729 90)
+		(layer "F.SilkS")
+		(effects
+			(font
+				(size 1 1)
+				(thickness 0.1)
+			)
+			(justify left bottom)
+		)
+	)
+	(gr_text "V"
+		(at 122 56.5 90)
+		(layer "F.SilkS")
+		(effects
+			(font
+				(size 1 1)
+				(thickness 0.1)
+			)
+			(justify left bottom)
+		)
+	)
+	(gr_text "T"
+		(at 124.5 56.5 90)
+		(layer "F.SilkS")
+		(effects
+			(font
+				(size 1 1)
+				(thickness 0.1)
+			)
+			(justify left bottom)
+		)
+	)
+	(gr_text "E"
+		(at 127 56.5 90)
+		(layer "F.SilkS")
+		(effects
+			(font
+				(size 1 1)
+				(thickness 0.1)
+			)
+			(justify left bottom)
+		)
+	)
+	(gr_text "G"
+		(at 131 56.5 90)
+		(layer "F.SilkS")
+		(effects
+			(font
+				(size 1 1)
+				(thickness 0.1)
+			)
+			(justify left bottom)
+		)
+	)
+	(gr_text "V"
+		(at 155.5 56.35 90)
+		(layer "F.SilkS")
+		(effects
+			(font
+				(size 1 1)
+				(thickness 0.1)
+			)
+			(justify left bottom)
+		)
+	)
+	(gr_text "G"
+		(at 158.5 56.5 90)
+		(layer "F.SilkS")
+		(effects
+			(font
+				(size 1 1)
+				(thickness 0.1)
+			)
+			(justify left bottom)
+		)
+	)
+	(gr_text "D"
+		(at 161 56.5 90)
+		(layer "F.SilkS")
+		(effects
+			(font
+				(size 1 1)
+				(thickness 0.1)
+			)
+			(justify left bottom)
+		)
+	)
